File: ESP-01_Flasher_Hardware/ESP-01_Flasher_Hardware.sch (KiCad schematic (older format))
At the start: 13 parts

Commit message: layout
Parts:
- removed J?: USB_B, symbol Connector:USB_B
- added J2: USB_A, ESP01_Library:USBA, symbol Connector:USB_A
- C1: renamed from C?; footprint (none) -> Capacitors_SMD:C_0603_HandSoldering
- D1, D2, D3: renamed from D?; footprint (none) -> LEDs:LED_0603_HandSoldering
- J1: renamed from J?; footprint (none) -> Socket_Strips:Socket_Strip_Angled_1x07_Pitch2.54mm
- R1, R2, R3: renamed from R?; footprint (none) -> Resistors_SMD:R_0603_HandSoldering
- SW1, SW2: renamed from SW?; footprint (none) -> Button_Switch_SMD:SW_SPST_TL3305A
- U1: renamed from U?; footprint (none) -> ESP01_Library:ESP8266-01
- U2: renamed from U?; footprint (none) -> Housings_SSOP:SSOP-28_5.3x10.2mm_Pitch0.65mm
Changed lines of the file:
@@
 $EndDescr
 $Comp
-L Project_Library:ESP-01 U?
+L Project_Library:ESP-01 U1
 U 1 1 5C2B985B
 P 6400 4550
-F 0 "U?" H 6700 5125 50  0000 C CNN
+F 0 "U1" H 6700 5125 50  0000 C CNN
 F 1 "ESP-01" H 6700 5034 50  0000 C CNN
-F 2 "" H 5950 4650 50  0001 C CNN
+F 2 "ESP01_Library:ESP8266-01" H 5950 4650 50  0001 C CNN
 F 3 "" H 5950 4650 50  0001 C CNN
 	1    6400 4550
@@
 $EndComp
 $Comp
-L Switch:SW_Push SW?
+L Switch:SW_Push SW1
 U 1 1 5C2B9946
 P 6300 2500
-F 0 "SW?" H 6300 2785 50  0000 C CNN
+F 0 "SW1" H 6300 2785 50  0000 C CNN
 F 1 "SW_Push" H 6300 2694 50  0000 C CNN
-F 2 "" H 6300 2700 50  0001 C CNN
+F 2 "Button_Switch_SMD:SW_SPST_TL3305A" H 6300 2700 50  0001 C CNN
 F 3 "" H 6300 2700 50  0001 C CNN
 	1    6300 2500
@@
 $EndComp
 $Comp
-L Switch:SW_Push SW?
+L Switch:SW_Push SW2
 U 1 1 5C2B9974
 P 6300 2750
-F 0 "SW?" H 6300 2700 50  0000 C CNN
+F 0 "SW2" H 6300 2700 50  0000 C CNN
 F 1 "SW_Push" H 6300 2600 50  0000 C CNN
-F 2 "" H 6300 2950 50  0001 C CNN
+F 2 "Button_Switch_SMD:SW_SPST_TL3305A" H 6300 2950 50  0001 C CNN
 F 3 "" H 6300 2950 50  0001 C CNN
 	1    6300 2750
-	1    0    0    -1
-$EndComp
-$Comp
-L Connector:USB_B J?
-U 1 1 5C2B9A7F
-P 7000 2700
-F 0 "J?" H 7055 3167 50  0000 C CNN
-F 1 "USB_B" H 7055 3076 50  0000 C CNN
-F 2 "" H 7150 2650 50  0001 C CNN
-F 3 " ~" H 7150 2650 50  0001 C CNN
-	1    7000 2700
 	1    0    0    -1
 $EndComp
@@
 	7300 2800 7350 2800
 $Comp
-L power:+5V #PWR?
+L power:+5V #PWR0101
 U 1 1 5C2B9CD0
 P 7350 2450
-F 0 "#PWR?" H 7350 2300 50  0001 C CNN
+F 0 "#PWR0101" H 7350 2300 50  0001 C CNN
 F 1 "+5V" H 7365 2623 50  0000 C CNN
 F 2 "" H 7350 2450 50  0001 C CNN
@@
 	7350 2500 7350 2450
 $Comp
-L power:GND #PWR?
+L power:GND #PWR0102
 U 1 1 5C2B9D27
 P 6950 3150
-F 0 "#PWR?" H 6950 2900 50  0001 C CNN
+F 0 "#PWR0102" H 6950 2900 50  0001 C CNN
 F 1 "GND" H 6955 2977 50  0000 C CNN
 F 2 "" H 6950 3150 50  0001 C CNN
@@
 	6950 3100 7000 3100
 $Comp
-L power:+5V #PWR?
+L power:+5V #PWR0103
 U 1 1 5C2DDD36
 P 8850 2400
-F 0 "#PWR?" H 8850 2250 50  0001 C CNN
+F 0 "#PWR0103" H 8850 2250 50  0001 C CNN
 F 1 "+5V" H 8865 2573 50  0000 C CNN
 F 2 "" H 8850 2400 50  0001 C CNN
@@
 NoConn ~ 8150 3500
 $Comp
-L Device:LED D?
+L Device:LED D1
 U 1 1 5C2DDF87
 P 9750 4000
-F 0 "D?" H 9900 4050 50  0000 R CNN
+F 0 "D1" H 9900 4050 50  0000 R CNN
 F 1 "Tx" H 9800 3900 50  0000 R CNN
-F 2 "" H 9750 4000 50  0001 C CNN
+F 2 "LEDs:LED_0603_HandSoldering" H 9750 4000 50  0001 C CNN
 F 3 "~" H 9750 4000 50  0001 C CNN
 	1    9750 4000
@@
 $EndComp
 $Comp
-L Device:R R?
+L Device:R R1
 U 1 1 5C2DDFFB
 P 9750 3650
-F 0 "R?" H 9820 3696 50  0000 L CNN
+F 0 "R1" H 9820 3696 50  0000 L CNN
 F 1 "330" V 9750 3550 50  0000 L CNN
-F 2 "" V 9680 3650 50  0001 C CNN
+F 2 "Resistors_SMD:R_0603_HandSoldering" V 9680 3650 50  0001 C CNN
 F 3 "~" H 9750 3650 50  0001 C CNN
 	1    9750 3650
@@
 $EndComp
 $Comp
-L Device:LED D?
+L Device:LED D2
 U 1 1 5C2DE1E7
 P 10000 4100
-F 0 "D?" H 10150 4150 50  0000 R CNN
+F 0 "D2" H 10150 4150 50  0000 R CNN
 F 1 "Rx" H 10050 4000 50  0000 R CNN
-F 2 "" H 10000 4100 50  0001 C CNN
+F 2 "LEDs:LED_0603_HandSoldering" H 10000 4100 50  0001 C CNN
 F 3 "~" H 10000 4100 50  0001 C CNN
 	1    10000 4100
@@
 $EndComp
 $Comp
-L Device:R R?
+L Device:R R2
 U 1 1 5C2DE1ED
 P 10000 3750
-F 0 "R?" H 10070 3796 50  0000 L CNN
+F 0 "R2" H 10070 3796 50  0000 L CNN
 F 1 "330" V 10000 3650 50  0000 L CNN
-F 2 "" V 9930 3750 50  0001 C CNN
+F 2 "Resistors_SMD:R_0603_HandSoldering" V 9930 3750 50  0001 C CNN
 F 3 "~" H 10000 3750 50  0001 C CNN
 	1    10000 3750
@@
 $EndComp
 $Comp
-L Device:LED D?
+L Device:LED D3
 U 1 1 5C2DE55F
 P 10250 4200
-F 0 "D?" H 10400 4250 50  0000 R CNN
+F 0 "D3" H 10400 4250 50  0000 R CNN
 F 1 "PWR" H 10300 4100 50  0000 R CNN
-F 2 "" H 10250 4200 50  0001 C CNN
+F 2 "LEDs:LED_0603_HandSoldering" H 10250 4200 50  0001 C CNN
 F 3 "~" H 10250 4200 50  0001 C CNN
 	1    10250 4200
@@
 $EndComp
 $Comp
-L Device:R R?
+L Device:R R3
 U 1 1 5C2DE565
 P 10250 3850
-F 0 "R?" H 10320 3896 50  0000 L CNN
+F 0 "R3" H 10320 3896 50  0000 L CNN
 F 1 "330" V 10250 3750 50  0000 L CNN
-F 2 "" V 10180 3850 50  0001 C CNN
+F 2 "Resistors_SMD:R_0603_HandSoldering" V 10180 3850 50  0001 C CNN
 F 3 "~" H 10250 3850 50  0001 C CNN
 	1    10250 3850
@@
 	10250 4350 10250 4550
 $Comp
-L power:GND #PWR?
+L power:GND #PWR0104
 U 1 1 5C2DEABE
 P 10250 4600
-F 0 "#PWR?" H 10250 4350 50  0001 C CNN
+F 0 "#PWR0104" H 10250 4350 50  0001 C CNN
 F 1 "GND" H 10255 4427 50  0000 C CNN
 F 2 "" H 10250 4600 50  0001 C CNN
@@
 Connection ~ 8950 4550
 $Comp
-L Project_Library:FT232RL U?
+L Project_Library:FT232RL U2
 U 1 1 5C2DDB5A
 P 8350 4350
-F 0 "U?" H 8875 6147 60  0000 C CNN
+F 0 "U2" H 8875 6147 60  0000 C CNN
 F 1 "FT232RL" H 8875 6041 60  0000 C CNN
-F 2 "" H 7800 4650 60  0001 C CNN
+F 2 "Housings_SSOP:SSOP-28_5.3x10.2mm_Pitch0.65mm" H 7800 4650 60  0001 C CNN
 F 3 "" H 7800 4650 60  0001 C CNN
 	1    8350 4350
@@
 	9600 3000 9650 3000
 $Comp
-L power:+3.3V #PWR?
+L power:+3.3V #PWR0105
 U 1 1 5C2E3340
 P 7900 2950
-F 0 "#PWR?" H 7900 2800 50  0001 C CNN
+F 0 "#PWR0105" H 7900 2800 50  0001 C CNN
 F 1 "+3.3V" H 7915 3123 50  0000 C CNN
 F 2 "" H 7900 2950 50  0001 C CNN
@@
 	7900 3000 7900 2950
 $Comp
-L Device:C C?
+L Device:C C1
 U 1 1 5C2E3A51
 P 7900 3150
-F 0 "C?" H 7750 3250 50  0000 L CNN
+F 0 "C1" H 7750 3250 50  0000 L CNN
 F 1 ".1uF" H 7700 3050 50  0000 L CNN
-F 2 "" H 7938 3000 50  0001 C CNN
+F 2 "Capacitors_SMD:C_0603_HandSoldering" H 7938 3000 50  0001 C CNN
 F 3 "~" H 7900 3150 50  0001 C CNN
 	1    7900 3150
@@
 Connection ~ 7900 3000
 $Comp
-L power:GND #PWR?
+L power:GND #PWR0106
 U 1 1 5C2E3C3D
 P 7900 3650
-F 0 "#PWR?" H 7900 3400 50  0001 C CNN
+F 0 "#PWR0106" H 7900 3400 50  0001 C CNN
 F 1 "GND" H 7905 3477 50  0000 C CNN
 F 2 "" H 7900 3650 50  0001 C CNN
@@
 Ylw
 $Comp
-L power:+3.3V #PWR?
+L power:+3.3V #PWR0107
 U 1 1 5C2EC5E6
 P 5800 4150
-F 0 "#PWR?" H 5800 4000 50  0001 C CNN
+F 0 "#PWR0107" H 5800 4000 50  0001 C CNN
 F 1 "+3.3V" H 5815 4323 50  0000 C CNN
 F 2 "" H 5800 4150 50  0001 C CNN
@@
 $EndComp
 $Comp
-L power:GND #PWR?
+L power:GND #PWR0108
 U 1 1 5C2ED1A4
 P 5800 4350
-F 0 "#PWR?" H 5800 4100 50  0001 C CNN
+F 0 "#PWR0108" H 5800 4100 50  0001 C CNN
 F 1 "GND" H 5805 4177 50  0000 C CNN
 F 2 "" H 5800 4350 50  0001 C CNN
@@
 	6550 2750 6550 2850
 $Comp
-L power:GND #PWR?
+L power:GND #PWR0109
 U 1 1 5C2F22F8
 P 6550 2850
-F 0 "#PWR?" H 6550 2600 50  0001 C CNN
+F 0 "#PWR0109" H 6550 2600 50  0001 C CNN
 F 1 "GND" H 6555 2677 50  0000 C CNN
 F 2 "" H 6550 2850 50  0001 C CNN
@@
 	5650 1750 5650 4850
 $Comp
-L Connector:Conn_01x07_Female J?
+L Connector:Conn_01x07_Female J1
 U 1 1 5C312C51
 P 5300 2700
-F 0 "J?" H 5327 2726 50  0000 L CNN
+F 0 "J1" H 5327 2726 50  0000 L CNN
 F 1 "Conn_01x07_Female" V 5450 2300 50  0000 L CNN
-F 2 "" H 5300 2700 50  0001 C CNN
+F 2 "Socket_Strips:Socket_Strip_Angled_1x07_Pitch2.54mm" H 5300 2700 50  0001 C CNN
 F 3 "~" H 5300 2700 50  0001 C CNN
 	1    5300 2700
@@
 $EndComp
 $Comp
-L power:GND #PWR?
+L power:GND #PWR0110
 U 1 1 5C312D44
 P 5050 3050
-F 0 "#PWR?" H 5050 2800 50  0001 C CNN
+F 0 "#PWR0110" H 5050 2800 50  0001 C CNN
 F 1 "GND" H 5055 2877 50  0000 C CNN
 F 2 "" H 5050 3050 50  0001 C CNN
@@
 	4500 2150 10400 2150
 $Comp
-L power:+5V #PWR?
+L power:+5V #PWR0111
 U 1 1 5C325788
 P 5050 2350
-F 0 "#PWR?" H 5050 2200 50  0001 C CNN
+F 0 "#PWR0111" H 5050 2200 50  0001 C CNN
 F 1 "+5V" H 5050 2500 50  0000 C CNN
 F 2 "" H 5050 2350 50  0001 C CNN
@@
 $EndComp
 $Comp
-L power:+3.3V #PWR?
+L power:+3.3V #PWR0112
 U 1 1 5C325870
 P 4900 2350
-F 0 "#PWR?" H 4900 2200 50  0001 C CNN
+F 0 "#PWR0112" H 4900 2200 50  0001 C CNN
 F 1 "+3.3V" H 4850 2500 50  0000 C CNN
 F 2 "" H 4900 2350 50  0001 C CNN
@@
 Wire Wire Line
 	5100 2500 4900 2500
+$Comp
+L Connector:USB_A J2
+U 1 1 5C19F1C7
+P 7000 2700
+F 0 "J2" H 7055 3167 50  0000 C CNN
+F 1 "USB_A" H 7055 3076 50  0000 C CNN
+F 2 "ESP01_Library:USBA" H 7150 2650 50  0001 C CNN
+F 3 " ~" H 7150 2650 50  0001 C CNN
+	1    7000 2700
+	1    0    0    -1
+$EndComp
 $EndSCHEMATC
